File: morgalo.kicad_pcb (KiCad board)
At the start: 2 copper layers, 25.7 x 21.5 mm, 11 parts, among them J1 USB_A, Q1 Q_NPN_BCE, Q2 Q_NPN_BCE

Commit message: Add files via upload
Routing:
- net Net-(D1-Pad2): track 30.4 -> 20.2 mm
- net Net-(C2-Pad2): track 30.9 -> 26.7 mm
- net Net-(C1-Pad1): track 21.8 -> 24.7 mm
- net Net-(D2-Pad1): track 7.00 -> 8.39 mm
- net Net-(J1-Pad4): track 41.8 -> 40.9 mm
- net Net-(C2-Pad1): track 12.5 -> 11.6 mm
Other:
- board size 25.7 x 21.5 mm -> 21.7 x 21.7 mm
- net class Default: trace_width 0.25 -> 0.6
- rule trace_min: 0.25 -> 0.6
